File: ブレッドボード_3/ブレッドボード_3.kicad_sch (KiCad schematic)
At the start: 11 parts, among them J1 Conn_01x12_Socket, J10 XIAO_Rudder, J11 XIAO_Under, J2 BNO055, J3 SD_0, J4 GPS, J5 Conn_01x12_Socket, J6 ICS, J7 Conn_01x08_Socket, J8 ICS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

Commit message: change Conn 5P to 6P
Parts:
- J10: footprint ブレッドボード_3:CONN5_B05B-PASK_JST -> ブレッドボード_3:CONN_B06B-PASK_JST; symbol Connector:Conn_01x05_Socket -> Connector:Conn_01x06_Socket
Connections:
- net 5V_DC_Rudder: now also J10.6 (Pin_6); no longer J10.5 (Pin_5)
- net DC_GND: now also J10.2 (Pin_2); no longer J10.1 (Pin_1)
- net EN_ICS: now also J10.3 (Pin_3); no longer J10.2 (Pin_2)
- net RX_ICS: now also J10.4 (Pin_4); no longer J10.3 (Pin_3)
- net SIG_ICS: now also J10.1 (Pin_1); no longer J1.11 (Pin_11)
- net TX_ICS: now also J10.5 (Pin_5); no longer J10.4 (Pin_4)
- net RX_ESP: now reaches J7.7 (Pin_7)
- net RX_ESP: now also J1.11 (Pin_11)
- no-connect marks 2 -> 1
Other:
- note removed: "RX_ESPは排除しました"
Changed lines of the file:
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@@
-		)
-	)
-	(text "RX_ESPは排除しました"
-		(exclude_from_sim no)
-		(at 210.566 137.668 0)
-		(effects
-			(font
-				(face "KiCad Font")
-				(size 2.54 2.54)
-				(thickness 0.508)
-				(bold yes)
-				(color 255 0 0 1)
-			)
 		)
 	)
@@
 		)
 	)
-	(text "RX_ESPは排除しました"
-		(exclude_from_sim no)
-		(at 78.232 115.57 0)
-		(effects
-			(font
-				(face "KiCad Font")
-				(size 2.54 2.54)
-				(thickness 0.508)
-				(bold yes)
-				(color 255 0 0 1)
-			)
-		)
-	)
 	(text "Bico"
 		(exclude_from_sim no)
@@
 			)
 		)
-	)
-	(no_connect
-		(at 180.34 135.89)
 	)
 	(no_connect
@@
 		)
 	)
+	(label "RX_ESP"
+		(at 180.34 135.89 0)
+		(effects
+			(font
+				(size 1.27 1.27)
+			)
+			(justify left bottom)
+		)
+	)
 	(label "RX_SD0"
 		(at 158.75 55.88 0)
@@
 		)
 	)
+	(label "SIG_ICS"
+		(at 260.35 20.32 180)
+		(effects
+			(font
+				(size 1.27 1.27)
+			)
+			(justify right bottom)
+		)
+	)
 	(label "SDA_AS0"
 		(at 60.96 129.54 180)
@@
 		)
 	)
-	(label "SIG_ICS"
-		(at 38.1 119.38 0)
-		(effects
-			(font
-				(size 1.27 1.27)
-			)
-			(justify left bottom)
-		)
-	)
 	(label "GND_BNO"
 		(at 127 21.59 0)
@@
 		)
 	)
+	(label "RX_ESP"
+		(at 38.1 119.38 0)
+		(effects
+			(font
+				(size 1.27 1.27)
+			)
+			(justify left bottom)
+		)
+	)
 	(label "SDA_BNO_BMP"
 		(at 38.1 129.54 0)
@@
 	)
 	(symbol
-		(lib_id "Connector:Conn_01x05_Socket")
-		(at 265.43 27.94 0)
+		(lib_id "Connector:Conn_01x06_Socket")
+		(at 265.43 25.4 0)
 		(unit 1)
 		(exclude_from_sim no)
@@
 		(fields_autoplaced yes)
 		(property "Reference" "J10"
-			(at 266.7 26.6699 0)
+			(at 266.7 25.3999 0)
 			(effects
 				(font
@@
 		)
 		(property "Value" "XIAO_Rudder"
-			(at 266.7 29.2099 0)
+			(at 266.7 27.9399 0)
 			(effects
 				(font
@@
 			)
 		)
-		(property "Footprint" "ブレッドボード_3:CONN5_B05B-PASK_JST"
-			(at 265.43 27.94 0)
+		(property "Footprint" "ブレッドボード_3:CONN_B06B-PASK_JST"
+			(at 265.43 25.4 0)
 			(effects
 				(font
@@
 		)
 		(property "Datasheet" "~"
-			(at 265.43 27.94 0)
+			(at 265.43 25.4 0)
 			(effects
 				(font
@@
 			)
 		)
-		(property "Description" "Generic connector, single row, 01x05, script generated"
-			(at 265.43 27.94 0)
+		(property "Description" "Generic connector, single row, 01x06, script generated"
+			(at 265.43 25.4 0)
 			(effects
 				(font
@@
 		(pin "5"
 		)
+		(pin "6"
+		)
 		(instances

Commit message: 家のPCで更新
Parts:
- added J12: SIG_ICS, ブレッドボード_3:CONN_B02B-PASK-1_JST, symbol Connector:Conn_01x02_Socket
- J10: footprint ブレッドボード_3:CONN_B06B-PASK_JST -> ブレッドボード_3:CONN_B05B-PASK_JST; symbol Connector:Conn_01x06_Socket -> Connector:Conn_01x05_Socket
Connections:
- net 5V_DC_Rudder: now also J10.5 (Pin_5); no longer J10.6 (Pin_6)
- net DC_GND: now also J10.1 (Pin_1); no longer J10.2 (Pin_2)
- net EN_ICS: now also J10.2 (Pin_2); no longer J10.3 (Pin_3)
- net RX_ICS: now also J10.3 (Pin_3); no longer J10.4 (Pin_4)
- net SIG_ICS: now also J12.1 (Pin_1), J12.2 (Pin_2); no longer J10.1 (Pin_1)
- net TX_ICS: now also J10.4 (Pin_4); no longer J10.5 (Pin_5)
Other:
- moved on the sheet: J11, J9
Changed lines of the file:
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@@
 		)
+	)
+	(junction
+		(at 256.54 29.21)
+		(diameter 0)
+		(color 0 0 0 0)
 	)
 	(no_connect
@@
 	(wire
 		(pts
-			(xy 257.81 46.99) (xy 264.16 46.99)
-		)
-		(stroke
-			(width 0)
-			(type default)
-		)
-	)
-	(wire
-		(pts
 			(xy 120.65 26.67) (xy 127 26.67)
 		)
@@
 	(wire
 		(pts
-			(xy 257.81 49.53) (xy 264.16 49.53)
-		)
-		(stroke
-			(width 0)
-			(type default)
-		)
-	)
-	(wire
-		(pts
 			(xy 149.86 50.8) (xy 158.75 50.8)
 		)
@@
 	(wire
 		(pts
-			(xy 264.16 41.91) (xy 257.81 41.91)
-		)
-		(stroke
-			(width 0)
-			(type default)
-		)
-	)
-	(wire
-		(pts
 			(xy 120.65 58.42) (xy 129.54 58.42)
 		)
@@
 	(wire
 		(pts
-			(xy 264.16 44.45) (xy 257.81 44.45)
+			(xy 254 29.21) (xy 256.54 29.21)
 		)
 		(stroke
@@
 		(pts
 			(xy 120.65 24.13) (xy 127 24.13)
+		)
+		(stroke
+			(width 0)
+			(type default)
+		)
+	)
+	(wire
+		(pts
+			(xy 256.54 26.67) (xy 256.54 29.21)
 		)
 		(stroke
@@
 	)
 	(label "DC_GND"
-		(at 257.81 58.42 180)
+		(at 256.54 68.58 180)
 		(effects
 			(font
@@
 	)
 	(label "SPK"
-		(at 257.81 55.88 180)
+		(at 256.54 66.04 180)
 		(effects
 			(font
@@
 	)
 	(label "DC_GND"
-		(at 257.81 41.91 180)
+		(at 256.54 52.07 180)
 		(effects
 			(font
@@
 	)
 	(label "TX_Under"
-		(at 257.81 46.99 180)
+		(at 256.54 57.15 180)
 		(effects
 			(font
@@
 	)
 	(label "TX_ICS"
-		(at 260.35 30.48 180)
+		(at 256.54 43.18 180)
 		(effects
 			(font
@@
 	)
 	(label "EN_ICS"
-		(at 260.35 25.4 180)
+		(at 256.54 38.1 180)
 		(effects
 			(font
@@
 	)
 	(label "5V_DC_Under"
-		(at 257.81 49.53 180)
+		(at 256.54 59.69 180)
 		(effects
 			(font
@@
 	)
 	(label "5V_DC_Rudder"
-		(at 260.35 33.02 180)
+		(at 256.54 45.72 180)
 		(effects
 			(font
@@
 	)
 	(label "RX_Under"
-		(at 257.81 44.45 180)
+		(at 256.54 54.61 180)
 		(effects
 			(font
@@
 	)
 	(label "DC_GND"
-		(at 260.35 22.86 180)
-		(effects
-			(font
-				(size 1.27 1.27)
-			)
-			(justify right bottom)
-		)
-	)
-	(label "SIG_ICS"
-		(at 260.35 20.32 180)
+		(at 256.54 35.56 180)
 		(effects
 			(font
@@
 	)
 	(label "RX_ICS"
-		(at 260.35 27.94 180)
+		(at 256.54 40.64 180)
 		(effects
 			(font
@@
 		)
 	)
+	(label "SIG_ICS"
+		(at 254 29.21 180)
+		(effects
+			(font
+				(size 1.27 1.27)
+			)
+			(justify right bottom)
+		)
+	)
 	(label "DC_GND"
 		(at 158.75 63.5 0)
@@
 	)
 	(symbol
-		(lib_id "Connector:Conn_01x06_Socket")
-		(at 265.43 25.4 0)
+		(lib_id "Connector:Conn_01x05_Socket")
+		(at 261.62 40.64 0)
 		(unit 1)
 		(exclude_from_sim no)
@@
 		(fields_autoplaced yes)
 		(property "Reference" "J10"
-			(at 266.7 25.3999 0)
+			(at 262.89 39.3699 0)
 			(effects
 				(font
@@
 		)
 		(property "Value" "XIAO_Rudder"
-			(at 266.7 27.9399 0)
+			(at 262.89 41.9099 0)
 			(effects
 				(font
@@
 			)
 		)
-		(property "Footprint" "ブレッドボード_3:CONN_B06B-PASK_JST"
-			(at 265.43 25.4 0)
+		(property "Footprint" "ブレッドボード_3:CONN_B05B-PASK_JST"
+			(at 261.62 40.64 0)
 			(effects
 				(font
@@
 		)
 		(property "Datasheet" "~"
-			(at 265.43 25.4 0)
-			(effects
-				(font
-					(size 1.27 1.27)
-				)
-				(hide yes)
-			)
-		)
-		(property "Description" "Generic connector, single row, 01x06, script generated"
-			(at 265.43 25.4 0)
+			(at 261.62 40.64 0)
+			(effects
+				(font
+					(size 1.27 1.27)
+				)
+				(hide yes)
+			)
+		)
+		(property "Description" "Generic connector, single row, 01x05, script generated"
+			(at 261.62 40.64 0)
 			(effects
 				(font
@@
 		)
 		(pin "5"
-		)
-		(pin "6"
 		)
 		(instances
@@
 	(symbol
 		(lib_id "Connector:Conn_01x02_Socket")
-		(at 262.89 55.88 0)
+		(at 261.62 26.67 0)
+		(unit 1)
+		(exclude_from_sim no)
+		(in_bom yes)
+		(on_board yes)
+		(dnp no)
+		(fields_autoplaced yes)
+		(property "Reference" "J12"
+			(at 262.89 26.6699 0)
+			(effects
+				(font
+					(size 1.27 1.27)
+				)
+				(justify left)
+			)
+		)
+		(property "Value" "SIG_ICS"
+			(at 262.89 29.2099 0)
+			(effects
+				(font
+					(size 1.27 1.27)
+				)
+				(justify left)
+			)
+		)
+		(property "Footprint" "ブレッドボード_3:CONN_B02B-PASK-1_JST"
+			(at 261.62 26.67 0)
+			(effects
+				(font
+					(size 1.27 1.27)
+				)
+				(hide yes)
+			)
+		)
+		(property "Datasheet" "~"
+			(at 261.62 26.67 0)
+			(effects
+				(font
+					(size 1.27 1.27)
+				)
+				(hide yes)
+			)
+		)
+		(property "Description" "Generic connector, single row, 01x02, script generated"
+			(at 261.62 26.67 0)
+			(effects
+				(font
+					(size 1.27 1.27)
+				)
+				(hide yes)
+			)
+		)
+		(pin "2"
+		)
+		(pin "1"
+		)
+		(instances
+			(project ""
+				(path "/ecdcb944-54ea-4e6c-a206-cc53d2130ed6"
+					(reference "J12")
+					(unit 1)
+				)
+			)
+		)
+	)
+	(symbol
+		(lib_id "Connector:Conn_01x02_Socket")
+		(at 261.62 66.04 0)
 		(unit 1)
 		(exclude_from_sim no)
@@
 		(fields_autoplaced yes)
 		(property "Reference" "J9"
-			(at 264.16 55.8799 0)
+			(at 262.89 66.0399 0)
 			(effects
 				(font
@@
 		)
 		(property "Value" "SPK"
-			(at 264.16 58.4199 0)
+			(at 262.89 68.5799 0)
 			(effects
 				(font
@@
 		)
 		(property "Footprint" "TORICA_Hardwarelib_self-made:PA_Connector_Post_2Pin"
-			(at 262.89 55.88 0)
+			(at 261.62 66.04 0)
 			(effects
 				(font
@@
 		)
 		(property "Datasheet" "~"
-			(at 262.89 55.88 0)
+			(at 261.62 66.04 0)
 			(effects
 				(font
@@
 		)
 		(property "Description" "Generic connector, single row, 01x02, script generated"
-			(at 262.89 55.88 0)
+			(at 261.62 66.04 0)
 			(effects
 				(font
@@
 	(symbol
 		(lib_id "Connector:Conn_01x04_Socket")
-		(at 269.24 44.45 0)
+		(at 261.62 54.61 0)
 		(unit 1)
 		(exclude_from_sim no)
@@
 		(dnp no)
 		(property "Reference" "J11"
-			(at 273.05 44.196 0)
+			(at 265.43 54.356 0)
 			(effects
 				(font
@@
 		)
 		(property "Value" "XIAO_Under"
-			(at 274.828 46.482 0)
+			(at 267.208 56.642 0)
 			(effects
 				(font
@@
 		)
 		(property "Footprint" "TORICA_Hardwarelib_self-made:PA_Connector_Pos_4Pin"
-			(at 269.24 44.45 0)
+			(at 261.62 54.61 0)
 			(effects
 				(font
@@
 		)
 		(property "Datasheet" "~"
-			(at 269.24 44.45 0)
+			(at 261.62 54.61 0)
 			(effects
 				(font
@@
 		)
 		(property "Description" "Generic connector, single row, 01x04, script generated"
-			(at 269.24 44.45 0)
-			(effects
-				(font
+			(at 261.62 54.61 0)
+			(effects
+				(font
