File: 各素子用/ICS/ICS.kicad_pcb (KiCad board)
At the start: 2 copper layers, 10.3 x 10.7 mm, 7 parts, among them J1 Conn_01x04_Socket, J2 Conn_01x03_Socket, U2 74AUC1G125, U3 74AUC1G125

Commit message: 家のPCで更新
Routing:
- net GND: track 9.24 -> 12.4 mm
